File: regulator.kicad_sch (KiCad schematic)
At the start: 37 parts, among them J6 39301022, Q1 NX7002BKW, U3 TPS7A8500RGRT, U4 TPSM82866AA0HRDMR, U5 TPS7A8500RGRT, U6 TPS259540DSGR

Commit message: Finish Regulator section
Parts:
- removed C12, C17, C19, C20, C24, C25, C27: 47u, Capacitor_SMD:C_0805_2012Metric, symbol Device:C_Small
- removed C13, C14, C31, C38: 0.1u, Capacitor_SMD:C_0805_2012Metric, symbol Device:C_Small
- removed C15: 0.01u, Capacitor_SMD:C_0805_2012Metric, symbol Device:C_Small
- removed C16, C18: 10u, Capacitor_SMD:C_0805_2012Metric, symbol Device:C_Small
- removed C33: 3.3n, Capacitor_SMD:C_0805_2012Metric, symbol Device:C_Small
- removed D1: GREEN, LED_SMD:LED_0805_2012Metric, symbol Device:LED
- removed L1: LSMGG160808T331RG, My Footprints:IND_LSMG_160808_TAY, symbol My Symbols:LSMGG160808T331RG
- removed R10: 10K, Resistor_SMD:R_0805_2012Metric, symbol Device:R_Small_US
- removed R27: 1K, Resistor_SMD:R_0805_2012Metric, symbol Device:R_Small_US
- removed R7: 205K, Resistor_SMD:R_0805_2012Metric, symbol Device:R_Small_US
- removed U3: TPS7A8500RGRT, My Footprints:QFN50P350X350X100-21N, symbol My Symbols:TPS7A8500RGRT
- removed U4: TPSM82866AA0HRDMR, My Footprints:RDM0023A-MFG, symbol My Symbols:TPSM82866AA0HRDMR
- removed U6: TPS259540DSGR, My Footprints:SON50P200X200X80-9N, symbol My Symbols:TPS259540DSGR
- added C44, C57, C58, C61: 10u, Capacitor_SMD:C_0805_2012Metric, symbol Device:C_Small
- added C46, C49, C50: 10uF, Capacitor_SMD:C_0603_1608Metric, symbol Device:C_Small
- added C47, C55: 0.1u, Capacitor_SMD:C_0805_2012Metric, symbol Device:C_Small
- added C48, C67: 2.2nF, Capacitor_SMD:C_0603_1608Metric, symbol Device:C_Small
- added C52: 4.7uF, Capacitor_SMD:C_1206_3216Metric, symbol Device:C_Small
- added C62: 4.7uF, Capacitor_SMD:C_0603_1608Metric, symbol Device:C_Small
- added C66, C68, C73, C76: 100u, Capacitor_SMD:C_0805_2012Metric, symbol Device:C_Small
- added D17: GREEN, LED_SMD:LED_0603_1608Metric, symbol Device:LED
- added L17: LSMGG160808T331RG, My Footprints:IND_LSMG_160808_TAY, symbol My Symbols:LSMGG160808T331RG
- added L18: 0.56u, My Footprints:COILCRAFT_XGL5050, symbol Device:L_Small
- added R103: 39.2K, Resistor_SMD:R_0603_1608Metric, symbol Device:R_Small_US
- added R104, R111: 49.9K, Resistor_SMD:R_0603_1608Metric, symbol Device:R_Small_US
- added R112: 1k, Resistor_SMD:R_0603_1608Metric, symbol Device:R_Small_US
- added R122: 2.21K, Resistor_SMD:R_0805_2012Metric, symbol Device:R_Small_US
- added R88, R90: 4.99K, Resistor_SMD:R_0603_1608Metric, symbol Device:R_Small_US
- added R89: 0, Resistor_SMD:R_0603_1608Metric, symbol Device:R_Small_US
- added R91: 33.2K, Resistor_SMD:R_0603_1608Metric, symbol Device:R_Small_US
- added R92: 47K, Resistor_SMD:R_0603_1608Metric, symbol Device:R_Small_US
- added R93: 49.9K, Resistor_SMD:R_0805_2012Metric, symbol Device:R_Small_US
- added TP5, TP6: ${SHORT_NET_NAME(1)}, TestPoint:TestPoint_THTPad_D2.0mm_Drill1.0mm, symbol Connector:TestPoint
- added U12: TPS259827ONRGET, My Footprints:TPS259827ONRGET, symbol My Symbols:TPS259827ONRGET
- added U7: LT3045xDD, Package_DFN_QFN:DFN-10-1EP_3x3mm_P0.5mm_EP1.65x2.38mm, symbol My Symbols:LT3045xDD
- added U8: LT8627SPJV-TRMPBF, My Footprints:05-08-7039_ADI, symbol My Symbols:LT8627SPJV-TRMPBF
- Q1: Cost 0.18 -> .1; MFG Nexperia -> Nexperia USA Inc.
- R86: renamed from R8; value 470 -> 182
- renumbered C32 to C65, C21 to C72, C23 to C74, C22 to C75, C26 to C77, C28 to C78, C29 to C79, C30 to C80, J6 to J7, L2 to L19, R9 to R85, U5 to U9
Connections:
- net +3.3V: now also C66.1, C68.1, C73.1, C76.1, L18.2, R103.1, TP6.1, U8.15 (OUTS)
- net +5.0V: now also C55.1, C58.1, C61.1, U7.10 (OUT), U7.9 (OUTS)
- net GND: now also C44.2, C46.2, C47.2, C48.2, C49.2, C50.2, C52.2, C55.2, C57.2, C58.2, C61.2, C62.2, C66.2, C67.2, C68.2, C73.2, C76.2, R104.2, R122.2, R89.2, R91.2, R92.2, R93.2, U12.10 (RETRY_DLY), U12.12 (LDSTRT), U12.14 (GND), U12.26 (GND), U12.4 (GND), U12.5 (GND), U7.11 (GND), U7.5 (ILIM), U7.8 (GND), U8.25 (GND), U8.26 (GND), U8.27 (GND), U8.28 (GND), U8.29 (GND), U8.3 (GND), U8.30 (GND), U8.31 (GND), U8.32 (GND), U8.4 (GND)
- net afe_pwrenb: now also U12.6 (EN/UVLO)
- net at Q1.3 (D): now also R112.2
- net at R86.1: now also U12.8 (ILIM)
- net +5VIN renamed +6VIN
- net +6VIN: now also U12.1 (IN), U12.16 (IN), U12.2 (IN), U12.25 (IN), U12.3 (IN)
- net PG renamed pg
- net pg: now also R111.2, U7.3 (EN/UV), U8.18 (PG)
- new net: C62.1, U8.11 (INTVCC)
- new net: C48.1, R90.2
- new net: R122.1, U12.9 (IMON)
- new net: R88.2, U8.10 (EN/UVLO)
- new net: C44.1, C47.1, L17.1, U7.1 (IN), U7.2 (IN), U7.6 (PGFB)
- new net: C57.1, R93.1, U7.7 (SET)
- new net: R89.1, U8.19 (SYNC)
- new net: TP5.1, U8.20 (CLKOUT)
- new net: D17.1 (K), R112.1
- new net +6.0V: C46.1, C49.1, C50.1, D17.2 (A), L17.2, R111.1, R88.1, U12.17 (OUT), U12.18 (OUT), U12.19 (OUT), U12.20 (OUT), U12.21 (OUT), U12.22 (OUT), U12.23 (OUT), U12.24 (OUT), U8.5 (PVIN), U8.6 (PVIN), U8.7 (PVIN), U8.8 (PVIN), U8.9 (SVIN)
- new net pgfb: C67.1, R103.2, R104.1, U8.16 (PGFB)
- new net rt: R92.1, U8.17 (RT)
- new net set: C52.1, R91.1, U8.13 (SET)
- new net sw: L18.1, U8.1 (SW), U8.2 (SW), U8.22 (SW), U8.23 (SW), U8.24 (SW)
- new net vc: R90.1, U8.14 (VC)
Other:
- note added: "15A Max"
- note added: "Add ADC to Rimon to measure current"
- note added: "DAC AVDD Regulator Sequences on after +3.3v"
- note added: "Install R89 for Pulse Skipping Mode Remove for Forced Continuous Mode"
- note added: "No Retry"
- note added: "Switching Frequency 2MHz"
- note removed: "545mA * (3.3v-2.5v) = 380mW"
- note removed: "ADC AVDD"
- moved on the sheet: C65, C72, C74, C75, C77, C78, C79, C80, J7, L19, R85, R86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

Commit message: Place SFP passives
Connections:
- net afe_pwrenb renamed PWR_ENB
- net pg: no longer names the net of Q1.1 (G), R111.2, U7.3 (EN/UV), U8.18 (PG)
Other:
- note added: "Logic Translator Regulator"
- moved on the sheet: D17, Q1, R111, R112
