File: sfp.kicad_sch (KiCad schematic)
At the start: 157 parts, among them J14 SFP+x8, U1 TCA9546A, U24 74LVC8T245, U25 TCA9546A, U9 74LVC8T245

Commit message: Finish Regulator section
Parts:
- renumbered C202 to C1, C211 to C10, C212 to C11, C213 to C12, C214 to C13, C215 to C14, C216 to C15, C217 to C16, C51 to C17, C52 to C18, C53 to C19, C203 to C2, C54 to C20, C55 to C21, C56 to C22, C57 to C23, C58 to C24, C59 to C25, C60 to C26, C61 to C27, C62 to C28, C63 to C29, C204 to C3, C64 to C30, C65 to C31, C66 to C32, C68 to C33, C219 to C34, C218 to C35, C67 to C36, C205 to C4, C206 to C5, C207 to C6, C208 to C7, C209 to C8, C210 to C9, D2 to D1, D5 to D10, D6 to D11, D7 to D12, D8 to D13, D9 to D14, D10 to D15, D11 to D16, D3 to D2, D12 to D3, D13 to D4, D14 to D5, D15 to D6, D16 to D7, D17 to D8, D4 to D9, J14 to J6, L8 to L1, L6 to L10, L7 to L11, L16 to L12, L17 to L13, L18 to L14, L19 to L15, L20 to L16, L9 to L2, L10 to L3, L11 to L4, L12 to L5, L13 to L6, L14 to L7, L15 to L8, L5 to L9, R110 to R1, R119 to R10, R120 to R11, R121 to R12, R122 to R13, R123 to R14, R124 to R15, R125 to R16, R126 to R17, R127 to R18, R128 to R19, R111 to R2, R129 to R20, R130 to R21, R131 to R22, R132 to R23, R133 to R24, R30 to R25, R31 to R26, R32 to R27, R33 to R28, R34 to R29, R112 to R3, R35 to R30, R36 to R31, R37 to R32, R38 to R33, R39 to R34, R40 to R35, R41 to R36, R42 to R37, R43 to R38, R44 to R39, R113 to R4, R45 to R40, R46 to R41, R47 to R42, R48 to R43, R49 to R44, R50 to R45, R51 to R46, R52 to R47, R53 to R48, R134 to R49, R114 to R5, R135 to R50, R136 to R51, R56 to R52, R54 to R53, R55 to R54, R65 to R55, R66 to R56, R67 to R57, R68 to R58, R69 to R59, R115 to R6, R70 to R60, R141 to R61, R142 to R62, R143 to R63, R144 to R64, R145 to R65, R146 to R66, R147 to R67, R148 to R68, R137 to R69, R116 to R7, R57 to R70, R138 to R71, R58 to R72, R139 to R73, R59 to R74, R140 to R75, R60 to R76, R149 to R77, R61 to R78, R150 to R79, R117 to R8, R62 to R80, R151 to R81, R63 to R82, R152 to R83, R64 to R84, R118 to R9, U9 to U1, U24 to U2, U25 to U3, U1 to U4
Connections:
- net SFP0.RX_N: now also J6.AL12 (RD-); no longer J6.AL19 (TD-)
- net SFP0.RX_P: now also J6.AL13 (RD+); no longer J6.AL18 (TD+)
- net SFP0.TX_N: now also J6.AL19 (TD-); no longer J6.AL12 (RD-)
- net SFP0.TX_P: now also J6.AL18 (TD+); no longer J6.AL13 (RD+)
- net SFP1.RX_N: now also J6.AT12 (RD-); no longer J6.AT19 (TD-)
- net SFP1.RX_P: now also J6.AT13 (RD+); no longer J6.AT18 (TD+)
- net SFP1.TX_N: now also J6.AT19 (TD-); no longer J6.AT12 (RD-)
- net SFP1.TX_P: now also J6.AT18 (TD+); no longer J6.AT13 (RD+)
- net SFP2.RX_N: now also J6.BL12 (RD-); no longer J6.BL19 (TD-)
- net SFP2.RX_P: now also J6.BL13 (RD+); no longer J6.BL18 (TD+)
- net SFP2.TX_N: now also J6.BL19 (TD-); no longer J6.BL12 (RD-)
- net SFP2.TX_P: now also J6.BL18 (TD+); no longer J6.BL13 (RD+)
- net SFP3.RX_N: now also J6.BT12 (RD-); no longer J6.BT19 (TD-)
- net SFP3.RX_P: now also J6.BT13 (RD+); no longer J6.BT18 (TD+)
- net SFP3.TX_N: now also J6.BT19 (TD-); no longer J6.BT12 (RD-)
- net SFP3.TX_P: now also J6.BT18 (TD+); no longer J6.BT13 (RD+)
- net SFP4.RX_N: now also J6.CL12 (RD-); no longer J6.CL19 (TD-)
- net SFP4.RX_P: now also J6.CL13 (RD+); no longer J6.CL18 (TD+)
- net SFP4.TX_N: now also J6.CL19 (TD-); no longer J6.CL12 (RD-)
- net SFP4.TX_P: now also J6.CL18 (TD+); no longer J6.CL13 (RD+)
- net SFP5.RX_N: now also J6.CT12 (RD-); no longer J6.CT19 (TD-)
- net SFP5.RX_P: now also J6.CT13 (RD+); no longer J6.CT18 (TD+)
- net SFP5.TX_N: now also J6.CT19 (TD-); no longer J6.CT12 (RD-)
- net SFP5.TX_P: now also J6.CT18 (TD+); no longer J6.CT13 (RD+)
- net SFP6.RX_N: now also J6.DL12 (RD-); no longer J6.DL19 (TD-)
- net SFP6.RX_P: now also J6.DL13 (RD+); no longer J6.DL18 (TD+)
- net SFP6.TX_N: now also J6.DL19 (TD-); no longer J6.DL12 (RD-)
- net SFP6.TX_P: now also J6.DL18 (TD+); no longer J6.DL13 (RD+)
- net SFP7.RX_N: now also J6.DT12 (RD-); no longer J6.DT19 (TD-)
- net SFP7.RX_P: now also J6.DT13 (RD+); no longer J6.DT18 (TD+)
- net SFP7.TX_N: now also J6.DT19 (TD-); no longer J6.DT12 (RD-)
- net SFP7.TX_P: now also J6.DT18 (TD+); no longer J6.DT13 (RD+)

Commit message: Place SFP passives
Connections:
- net I2C0.SCL: no longer R49.2, U3.14 (SCL)
- net I2C0.SDA: no longer R50.2, U3.15 (SDA)
- new net I2C.SCL: R49.2, U3.14 (SCL)
- new net I2C.SDA: R50.2, U3.15 (SDA)
Other:
- note added: "FPGA pulls TX_DIS low to enable SFP (Turns on Green LED) MOD_ABS is pulled low when module installed RX_LOS is pulled high when optical power is too low RED LED goes on when MOD_ABS is low and RX_LOS is high"
Changed lines of the file:
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@@
 	(text "ADDR 0x70"
 		(exclude_from_sim no)
-		(at 297.18 48.26 0)
+		(at 305.816 57.15 0)
 		(effects
 			(font
@@
 		)
 	)
+	(text "FPGA pulls TX_DIS low to enable SFP  (Turns on Green LED)\nMOD_ABS is pulled low when module installed\nRX_LOS is pulled high when optical power is too low\nRED LED goes on when MOD_ABS is low and RX_LOS is high"
+		(exclude_from_sim no)
+		(at 50.8 26.162 0)
+		(effects
+			(font
+				(size 1.27 1.27)
+			)
+			(justify left)
+		)
+	)
 	(text "ADDR 0x50, 0x51"
 		(exclude_from_sim no)
@@
 		)
 	)
-	(label "I2C0.SCL"
+	(label "I2C.SCL"
 		(at 317.5 44.45 0)
 		(effects
@@
 		)
 	)
-	(label "I2C0.SDA"
+	(label "I2C.SDA"
 		(at 317.5 46.99 0)
 		(effects
@@
 		)
 	)
-	(hierarchical_label "I2C0{SDA,SCL}"
+	(hierarchical_label "I2C{SDA,SCL}"
 		(shape bidirectional)
 		(at 312.42 41.91 180)
