File: cc-afe.kicad_pcb (KiCad board)
At the start: 6 copper layers, 241.3 x 170.4 mm, 270 parts, among them J1 6469028-1, J11 EPY.00.250.NTN, J12 0875-1G2T-V5, J13 EPY.00.250.NTN, J14 SFP+x8, J2 6469028-1, J3 6469028-1, J4 6469028-1, J5 6469028-1, J6 39301022, Q1 NX7002BKW, U1 TCA9546A, U2 DP83849CVS_NOPB, U24 74LVC8T245, U25 TCA9546A, U3 TPS7A8500RGRT, U4 TPSM82866AA0HRDMR, U5 TPS7A8500RGRT, U6 TPS259540DSGR, U7 AD5754BREZ, U8 SN74AVC8T245PW, U9 74LVC8T245, X1 CB3LV-3I-25M0000

Commit message: Finish Regulator section
Parts:
- removed the C12 at (294.6, 351.3)
- removed the C13 at (294.6, 349.0)
- removed the C14 at (294.6, 353.6)
- removed the C15 at (283.9, 353.0)
- removed the C16 at (287.8, 347.0)
- removed the C17 at (278.6, 320.9)
- removed the C18 at (285.6, 347.0)
- removed the C19 at (276.4, 320.9)
- removed the C20 at (282.9, 349.9)
- removed the C24 at (265.9, 322.1)
- removed the C25 at (263.6, 322.1)
- removed the C27 at (261.3, 322.1)
- removed the C31 at (294.6, 344.9)
- removed the C33 at (285.4, 324.8)
- removed C38: 0.1u, Capacitor_SMD:C_0805_2012Metric
- removed the D1 at (282.7, 315.2)
- removed the L1 at (294.5, 347.0)
- removed the R10 at (273.1, 315.7)
- removed the R27 at (280.1, 315.1)
- removed the R7 at (269.6, 316.0)
- removed the U3 at (288.8, 352.8)
- removed the U4 at (269.9, 320.7)
- removed the U6 at (283.7, 320.2)
- added C44: 10u, Capacitor_SMD:C_0805_2012Metric, F.Cu at (203.8, 190.4)
- added C46: 10uF, Capacitor_SMD:C_0603_1608Metric, F.Cu at (261.9, 241.5)
- added C47: 0.1u, Capacitor_SMD:C_0805_2012Metric, F.Cu at (203.8, 193.4)
- added C48: 2.2nF, Capacitor_SMD:C_0603_1608Metric, F.Cu at (261.9, 244.0)
- added C49: 10uF, Capacitor_SMD:C_0603_1608Metric, F.Cu at (261.9, 246.5)
- added C50: 10uF, Capacitor_SMD:C_0603_1608Metric, F.Cu at (261.9, 249.0)
- added C52: 4.7uF, Capacitor_SMD:C_1206_3216Metric, F.Cu at (280.4, 256.9)
- added C55: 0.1u, Capacitor_SMD:C_0805_2012Metric, F.Cu at (203.8, 196.4)
- added C57: 10u, Capacitor_SMD:C_0805_2012Metric, F.Cu at (203.8, 199.4)
- added C58: 10u, Capacitor_SMD:C_0805_2012Metric, F.Cu at (203.8, 202.4)
- added C61: 10u, Capacitor_SMD:C_0805_2012Metric, F.Cu at (208.3, 190.4)
- added C62: 4.7uF, Capacitor_SMD:C_0603_1608Metric, F.Cu at (261.9, 251.5)
- added C66: 100u, Capacitor_SMD:C_0805_2012Metric, F.Cu at (278.6, 244.7)
- added C67: 2.2nF, Capacitor_SMD:C_0603_1608Metric, F.Cu at (261.9, 254.0)
- added C68: 100u, Capacitor_SMD:C_0805_2012Metric, F.Cu at (278.6, 247.7)
- added C73: 100u, Capacitor_SMD:C_0805_2012Metric, F.Cu at (278.6, 250.8)
- added C76: 100u, Capacitor_SMD:C_0805_2012Metric, F.Cu at (278.6, 253.8)
- added D17: GREEN, LED_SMD:LED_0603_1608Metric, F.Cu at (282.8, 253.7)
- added L17: LSMGG160808T331RG, My Footprints:IND_LSMG_160808_TAY, F.Cu at (199.4, 198.1)
- added L18: 0.56u, My Footprints:COILCRAFT_XGL5050, F.Cu at (246.5, 248.8)
- added R103: 39.2K, Resistor_SMD:R_0603_1608Metric, F.Cu at (269.9, 241.5)
- added R104: 49.9K, Resistor_SMD:R_0603_1608Metric, F.Cu at (269.9, 244.0)
- added R111: 49.9K, Resistor_SMD:R_0603_1608Metric, F.Cu at (269.9, 246.5)
- added R112: 1k, Resistor_SMD:R_0603_1608Metric, F.Cu at (269.9, 249.0)
- added R122: 2.21K, Resistor_SMD:R_0805_2012Metric, F.Cu at (273.0, 309.6)
- added R88: 4.99K, Resistor_SMD:R_0603_1608Metric, F.Cu at (265.9, 244.0)
- added R89: 0, Resistor_SMD:R_0603_1608Metric, F.Cu at (265.9, 246.5)
- added R90: 4.99K, Resistor_SMD:R_0603_1608Metric, F.Cu at (265.9, 249.0)
- added R91: 33.2K, Resistor_SMD:R_0603_1608Metric, F.Cu at (265.9, 251.5)
- added R92: 47K, Resistor_SMD:R_0603_1608Metric, F.Cu at (265.9, 254.0)
- added R93: 49.9K, Resistor_SMD:R_0805_2012Metric, F.Cu at (198.9, 200.9)
- added TP5: Net-(U8-CLKOUT), TestPoint:TestPoint_THTPad_D2.0mm_Drill1.0mm, F.Cu at (282.8, 242.2)
- added TP6: +3.3V, TestPoint:TestPoint_THTPad_D2.0mm_Drill1.0mm, F.Cu at (282.8, 246.3)
- added U12: TPS259827ONRGET, My Footprints:TPS259827ONRGET, F.Cu at (274.7, 305.1)
- added U7: LT3045xDD, Package_DFN_QFN:DFN-10-1EP_3x3mm_P0.5mm_EP1.65x2.38mm, F.Cu at (198.9, 194.2)
- added U8: LT8627SPJV-TRMPBF, My Footprints:05-08-7039_ADI, F.Cu at (253.3, 248.6)
- R86: renamed from R8; value 470 -> 182
- moved C80 88.3 mm to (264.7, 277.0)
- moved C65 88.3 mm to (276.5, 271.2)
- moved C72 88.3 mm to (276.5, 275.4)
- moved C74 88.3 mm to (276.5, 279.9)
- moved C75 88.3 mm to (276.5, 277.6)
- moved C77 88.3 mm to (265.5, 279.8)
- moved C78 88.3 mm to (267.6, 274.1)
- moved C79 88.3 mm to (269.7, 274.1)
- moved L19 88.3 mm to (276.3, 273.3)
- moved U9 88.3 mm to (270.7, 279.3)
- moved Q1 58.9 mm to (266.9, 257.2)
- moved J2 25.4 mm to (166.8, 321.3)
- moved J3 25.4 mm to (192.2, 321.3)
- moved J7 14.3 mm to (293.8, 305.4)
- moved R85 14.3 mm to (285.4, 315.8)
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- renumbered C202 to C1, C211 to C10, C212 to C11, C213 to C12, C214 to C13, C215 to C14, C216 to C15, C217 to C16, C51 to C17, C52 to C18, C53 to C19, C203 to C2, C54 to C20, C55 to C21, C56 to C22, C57 to C23, C58 to C24, C59 to C25, C60 to C26, C61 to C27, C62 to C28, C63 to C29, C204 to C3, C64 to C30, C65 to C31, C66 to C32, C68 to C33, C219 to C34, C218 to C35, C67 to C36, C40 to C37, C11 to C39, C205 to C4, C34 to C40, C35 to C41, C36 to C42, C37 to C43, C39 to C45, C206 to C5, C9 to C51, C10 to C53, C5 to C54, C6 to C56, C7 to C59, C207 to C6, C8 to C60, C1 to C63, C3 to C64, C32 to C65, C208 to C7, C2 to C70, C4 to C71, C21 to C72, C23 to C74, C22 to C75, C26 to C77, C28 to C78, C29 to C79, C209 to C8, C30 to C80, C45 to C81, C46 to C82, C41 to C83, C42 to C84, C44 to C85, C43 to C86, C47 to C87, C48 to C88, C49 to C89, C210 to C9, C50 to C90, D2 to D1, D5 to D10, D6 to D11, D7 to D12, D8 to D13, D9 to D14, D10 to D15, D11 to D16, D3 to D2, D12 to D3, D13 to D4, D14 to D5, D15 to D6, D16 to D7, D17 to D8, D4 to D9, J13 to J10, J14 to J6, J6 to J7, J12 to J8, J11 to J9, L8 to L1, L6 to L10, L7 to L11, L16 to L12, L17 to L13, L18 to L14, L19 to L15, L20 to L16, L2 to L19, L9 to L2, L3 to L20, L4 to L21, L10 to L3, L11 to L4, L12 to L5, L13 to L6, L14 to L7, L15 to L8, L5 to L9, MT5 to MT4, MT7 to MT5, MT8 to MT6, R110 to R1, R119 to R10, R6 to R100, R17 to R101, R15 to R102, R3 to R105, R11 to R106, R4 to R107, R12 to R108, R18 to R109, R120 to R11, R16 to R110, R14 to R113, R13 to R114, R19 to R115, R20 to R116, R25 to R118, R26 to R119, R121 to R12, R28 to R120, R29 to R121, R122 to R13, R123 to R14, R124 to R15, R125 to R16, R126 to R17, R127 to R18, R128 to R19, R111 to R2, R129 to R20, R130 to R21, R131 to R22, R132 to R23, R133 to R24, R30 to R25, R31 to R26, R32 to R27, R33 to R28, R34 to R29, R112 to R3, R35 to R30, R36 to R31, R37 to R32, R38 to R33, R39 to R34, R40 to R35, R41 to R36, R42 to R37, R43 to R38, R44 to R39, R113 to R4, R45 to R40, R46 to R41, R47 to R42, R48 to R43, R49 to R44, R50 to R45, R51 to R46, R52 to R47, R53 to R48, R134 to R49, R114 to R5, R135 to R50, R136 to R51, R56 to R52, R54 to R53, R55 to R54, R65 to R55, R66 to R56, R67 to R57, R68 to R58, R69 to R59, R115 to R6, R70 to R60, R141 to R61, R142 to R62, R143 to R63, R144 to R64, R145 to R65, R146 to R66, R147 to R67, R148 to R68, R137 to R69, R116 to R7, R57 to R70, R138 to R71, R58 to R72, R139 to R73, R59 to R74, R140 to R75, R60 to R76, R149 to R77, R61 to R78, R150 to R79, R117 to R8, R62 to R80, R151 to R81, R63 to R82, R152 to R83, R64 to R84, R9 to R85, R24 to R87, R118 to R9, R21 to R94, R22 to R95, R23 to R96, R1 to R97, R5 to R98, R2 to R99, U9 to U1, U8 to U10, U7 to U11, U24 to U2, U25 to U3, U1 to U4, U2 to U6, U5 to U9
Connections:
- J1 pad A2: unconnected-(J1-PadA2) -> /SFP/SFP4.TX_P
- J1 pad A3: unconnected-(J1-PadA3) -> /SFP/SFP5.TX_P
- J1 pad A4: unconnected-(J1-PadA4) -> /SFP/SFP6.TX_P
- J1 pad A5: unconnected-(J1-PadA5) -> /SFP/SFP7.TX_P
- J1 pad B2: unconnected-(J1-PadB2) -> /SFP/SFP4.TX_N
- J1 pad B3: unconnected-(J1-PadB3) -> /SFP/SFP5.TX_N
- J1 pad B4: unconnected-(J1-PadB4) -> /SFP/SFP6.TX_N
- J1 pad B5: unconnected-(J1-PadB5) -> /SFP/SFP7.TX_N
- J1 pad C2: unconnected-(J1-PadC2) -> /SFP/SFP4.RX_P
- J1 pad C3: unconnected-(J1-PadC3) -> /SFP/SFP5.RX_P
- J1 pad C4: unconnected-(J1-PadC4) -> /SFP/SFP6.RX_P
- J1 pad C5: unconnected-(J1-PadC5) -> /SFP/SFP7.RX_P
- J1 pad D2: unconnected-(J1-PadD2) -> /SFP/SFP4.RX_N
- J1 pad D3: unconnected-(J1-PadD3) -> /SFP/SFP5.RX_N
- J1 pad D4: unconnected-(J1-PadD4) -> /SFP/SFP6.RX_N
- J1 pad D5: unconnected-(J1-PadD5) -> /SFP/SFP7.RX_N
- J3 pad A6: unconnected-(J3-PadA6) -> /SFP/SFP0.TX_P
- J3 pad A7: unconnected-(J3-PadA7) -> /SFP/SFP1.TX_P
- J3 pad A8: unconnected-(J3-PadA8) -> /SFP/SFP2.TX_P
- J3 pad A9: unconnected-(J3-PadA9) -> /SFP/SFP3.TX_P
- J3 pad B6: unconnected-(J3-PadB6) -> /SFP/SFP0.TX_N
- J3 pad B7: unconnected-(J3-PadB7) -> /SFP/SFP1.TX_N
- J3 pad B8: unconnected-(J3-PadB8) -> /SFP/SFP2.TX_N
- J3 pad B9: unconnected-(J3-PadB9) -> /SFP/SFP3.TX_N
- J3 pad C6: unconnected-(J3-PadC6) -> /SFP/SFP0.RX_P
- J3 pad C7: unconnected-(J3-PadC7) -> /SFP/SFP1.RX_P
- J3 pad C8: unconnected-(J3-PadC8) -> /SFP/SFP2.RX_P
- J3 pad C9: unconnected-(J3-PadC9) -> /SFP/SFP3.RX_P
- J3 pad D6: unconnected-(J3-PadD6) -> /SFP/SFP0.RX_N
- J3 pad D7: unconnected-(J3-PadD7) -> /SFP/SFP1.RX_N
- J3 pad D8: unconnected-(J3-PadD8) -> /SFP/SFP2.RX_N
- J3 pad D9: unconnected-(J3-PadD9) -> /SFP/SFP3.RX_N
- J6 pad AL12: /SFP/SFP0.TX_N -> /SFP/SFP0.RX_N
- J6 pad AL13: /SFP/SFP0.TX_P -> /SFP/SFP0.RX_P
- J6 pad AL18: /SFP/SFP0.RX_P -> /SFP/SFP0.TX_P
- J6 pad AL19: /SFP/SFP0.RX_N -> /SFP/SFP0.TX_N
- J6 pad AT12: /SFP/SFP1.TX_N -> /SFP/SFP1.RX_N
- J6 pad AT13: /SFP/SFP1.TX_P -> /SFP/SFP1.RX_P
- J6 pad AT18: /SFP/SFP1.RX_P -> /SFP/SFP1.TX_P
- J6 pad AT19: /SFP/SFP1.RX_N -> /SFP/SFP1.TX_N
- J6 pad BL12: /SFP/SFP2.TX_N -> /SFP/SFP2.RX_N
- J6 pad BL13: /SFP/SFP2.TX_P -> /SFP/SFP2.RX_P
- J6 pad BL18: /SFP/SFP2.RX_P -> /SFP/SFP2.TX_P
- J6 pad BL19: /SFP/SFP2.RX_N -> /SFP/SFP2.TX_N
- J6 pad BT12: /SFP/SFP3.TX_N -> /SFP/SFP3.RX_N
- J6 pad BT13: /SFP/SFP3.TX_P -> /SFP/SFP3.RX_P
- J6 pad BT18: /SFP/SFP3.RX_P -> /SFP/SFP3.TX_P
- J6 pad BT19: /SFP/SFP3.RX_N -> /SFP/SFP3.TX_N
- J6 pad CL12: /SFP/SFP4.TX_N -> /SFP/SFP4.RX_N
- J6 pad CL13: /SFP/SFP4.TX_P -> /SFP/SFP4.RX_P
- J6 pad CL18: /SFP/SFP4.RX_P -> /SFP/SFP4.TX_P
- J6 pad CL19: /SFP/SFP4.RX_N -> /SFP/SFP4.TX_N
- J6 pad CT12: /SFP/SFP5.TX_N -> /SFP/SFP5.RX_N
- J6 pad CT13: /SFP/SFP5.TX_P -> /SFP/SFP5.RX_P
- J6 pad CT18: /SFP/SFP5.RX_P -> /SFP/SFP5.TX_P
- J6 pad CT19: /SFP/SFP5.RX_N -> /SFP/SFP5.TX_N
- J6 pad DL12: /SFP/SFP6.TX_N -> /SFP/SFP6.RX_N
- J6 pad DL13: /SFP/SFP6.TX_P -> /SFP/SFP6.RX_P
- J6 pad DL18: /SFP/SFP6.RX_P -> /SFP/SFP6.TX_P
- J6 pad DL19: /SFP/SFP6.RX_N -> /SFP/SFP6.TX_N
- J6 pad DT12: /SFP/SFP7.TX_N -> /SFP/SFP7.RX_N
- J6 pad DT13: /SFP/SFP7.TX_P -> /SFP/SFP7.RX_P
- J6 pad DT18: /SFP/SFP7.RX_P -> /SFP/SFP7.TX_P
- J6 pad DT19: /SFP/SFP7.RX_N -> /SFP/SFP7.TX_N
- J7 pad 2: /Regulators/+5VIN -> /Regulators/+6VIN
- Q1 pad 1: /Regulators/PG -> /Regulators/pg
Routing:
- net /Regulators/afe_pwrenb: track 120.5 -> 21.1 mm, vias 1 -> 0
- net GND: track 25.2 -> 3.10 mm
- net /Regulators/PG: track 8.53 -> 0.00 mm
- net +5.0V: track 7.86 -> 0.00 mm
- net Net-(U12-ILIM): track 4.48 -> 0.00 mm
- net Net-(U3-FB): track 3.70 -> 0.00 mm
- net Net-(U3-NR/SS): track 3.48 -> 0.00 mm
- net Net-(U6-DVDT): track 3.47 -> 0.00 mm
- net Net-(U4-VSET_MODE): track 3.08 -> 0.00 mm
- net Net-(Q1-D): track 2.77 -> 0.00 mm
- net Net-(D1-K) (its old number): track 2.62 -> 0.00 mm
- removed copper zone on F.Cu, net +3.3V
- removed copper zone on F.Cu, net +5.0V
- removed copper zone on F.Cu, net /Regulators/+3.3v_U3
- removed copper zone on F.Cu, net /Regulators/+5VIN
- removed copper zone on F.Cu, net GND

Commit message: Place SFP passives
Parts:
- C1, C10, C13, C14, C17, C18, C2, C21, C22, C25, C26, C29, C30, C33, C34, C35, C36, C5, C6, C81, C82, C83, C84, C85, C86, C9, L1, L10, L13, L14, L2, L5, L6, L9: moved to B.Cu
- moved G*** 119.2 mm to (201.4, 243.1)
- moved R53 42.0 mm to (73.6, 207.0)
- moved R54 42.0 mm to (73.6, 209.5)
- moved R55 42.0 mm to (77.6, 209.5)
- moved R56 42.0 mm to (77.6, 212.0)
- moved R57 42.0 mm to (77.6, 214.5)
- moved R58 42.0 mm to (77.6, 217.1)
- moved R59 42.0 mm to (77.6, 219.6)
- moved R60 42.0 mm to (77.6, 222.1)
- moved D3 40.6 mm to (83.5, 210.6)
- moved D4 40.6 mm to (83.5, 213.2)
- moved D5 40.6 mm to (83.5, 215.8)
- moved D6 40.6 mm to (83.5, 218.4)
- moved D7 40.6 mm to (83.5, 221.0)
- moved D8 40.6 mm to (83.5, 223.6)
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Connections:
- net /Regulators/afe_pwrenb renamed /Regulators/PWR_ENB
- net /Regulators/pg renamed Net-(Q1-G)
- J2 pad A10: unconnected-(J2-PadA10) -> /SFP/SFP_MOD_ABS6
- J2 pad A4: unconnected-(J2-PadA4) -> /SFP/SFP_TX_DIS0
- J2 pad A5: unconnected-(J2-PadA5) -> /SFP/SFP_TX_DIS4
- J2 pad A7: unconnected-(J2-PadA7) -> /SFP/SFP_RX_LOS3
- J2 pad A8: unconnected-(J2-PadA8) -> /SFP/SFP_RX_LOS7
- J2 pad A9: unconnected-(J2-PadA9) -> /SFP/SFP_MOD_ABS2
- J2 pad B10: unconnected-(J2-PadB10) -> /SFP/SFP_MOD_ABS7
- J2 pad B4: unconnected-(J2-PadB4) -> /SFP/SFP_TX_DIS1
- J2 pad B5: unconnected-(J2-PadB5) -> /SFP/SFP_TX_DIS5
- J2 pad B6: unconnected-(J2-PadB6) -> /SFP/SFP_RX_LOS0
- J2 pad B7: unconnected-(J2-PadB7) -> /SFP/SFP_RX_LOS4
- J2 pad B9: unconnected-(J2-PadB9) -> /SFP/SFP_MOD_ABS3
- J2 pad C4: unconnected-(J2-PadC4) -> /SFP/SFP_TX_DIS2
- J2 pad C5: unconnected-(J2-PadC5) -> /SFP/SFP_TX_DIS6
- J2 pad C6: unconnected-(J2-PadC6) -> /SFP/SFP_RX_LOS1
- J2 pad C7: unconnected-(J2-PadC7) -> /SFP/SFP_RX_LOS5
- J2 pad C8: unconnected-(J2-PadC8) -> /SFP/SFP_MOD_ABS0
- J2 pad C9: unconnected-(J2-PadC9) -> /SFP/SFP_MOD_ABS4
- J2 pad D4: unconnected-(J2-PadD4) -> /SFP/SFP_TX_DIS3
- J2 pad D5: unconnected-(J2-PadD5) -> /SFP/SFP_TX_DIS7
- J2 pad D6: unconnected-(J2-PadD6) -> /SFP/SFP_RX_LOS2
- J2 pad D7: unconnected-(J2-PadD7) -> /SFP/SFP_RX_LOS6
- J2 pad D8: unconnected-(J2-PadD8) -> /SFP/SFP_MOD_ABS1
- J2 pad D9: unconnected-(J2-PadD9) -> /SFP/SFP_MOD_ABS5
- J5 pad C10: /zuDFE Connectors/i2c_sda -> /SFP/I2C.SDA
- J5 pad C9: unconnected-(J5-PadC9) -> /SDI/MDIO
- J5 pad D10: /zuDFE Connectors/i2c_scl -> /SFP/I2C.SCL
- J5 pad D9: unconnected-(J5-PadD9) -> /SDI/MDC
- R49 pad 2: /SFP/I2C0.SCL -> /SFP/I2C.SCL
- R50 pad 2: /SFP/I2C0.SDA -> /SFP/I2C.SDA
- R87 pad 2: Net-(U6-MDIO) -> /SDI/MDIO
- U3 pad 14: /SFP/I2C0.SCL -> /SFP/I2C.SCL
- U3 pad 15: /SFP/I2C0.SDA -> /SFP/I2C.SDA
- U6 pad 66: Net-(U6-MDIO) -> /SDI/MDIO
- U6 pad 67: unconnected-(U6-MDC-Pad67) -> /SDI/MDC
Routing:
- net /Regulators/PWR_ENB: track 21.1 -> 0.00 mm

Commit message: Add digital Outputs
Parts:
- added C100: 1u, Capacitor_SMD:C_0603_1608Metric, F.Cu at (166.3, 216.2)
- added C101: 0.1u, Capacitor_SMD:C_0603_1608Metric, F.Cu at (166.3, 218.7)
- added C38: 0.1u, Capacitor_SMD:C_0603_1608Metric, B.Cu at (174.8, 192.8)
- added C69: 0.1u, Capacitor_SMD:C_0603_1608Metric, B.Cu at (174.8, 195.3)
- added C91: 0.1u, Capacitor_SMD:C_0603_1608Metric, B.Cu at (185.4, 194.5)
- added C92: 0.1u, Capacitor_SMD:C_0603_1608Metric, B.Cu at (185.4, 197.0)
- added C93: 0.1u, Capacitor_SMD:C_0603_1608Metric, B.Cu at (195.0, 192.0)
- added C94: 0.1u, Capacitor_SMD:C_0603_1608Metric, B.Cu at (207.2, 192.0)
- added C95: 0.1u, Capacitor_SMD:C_0603_1608Metric, B.Cu at (195.3, 193.5)
- added C96: 0.1u, Capacitor_SMD:C_0603_1608Metric, B.Cu at (207.2, 193.8)
- added C97: 0.1u, Capacitor_SMD:C_0603_1608Metric, F.Cu at (166.3, 208.7)
- added C98: 0.1u, Capacitor_SMD:C_0603_1608Metric, F.Cu at (166.3, 211.2)
- added C99: 1u, Capacitor_SMD:C_0603_1608Metric, F.Cu at (166.3, 213.7)
- added J11: EPY.00.250.NTN, My Footprints:LEMO_EPY.00.250.NTN, F.Cu at (173.7, 177.5)
- added J12: EPY.00.250.NTN, My Footprints:LEMO_EPY.00.250.NTN, F.Cu at (183.7, 177.5)
- added J13: EPY.00.250.NTN, My Footprints:LEMO_EPY.00.250.NTN, F.Cu at (193.7, 177.5)
- added J14: EPY.00.250.NTN, My Footprints:LEMO_EPY.00.250.NTN, F.Cu at (203.7, 177.5)
- added J15: EPY.00.250.NTN, My Footprints:LEMO_EPY.00.250.NTN, F.Cu at (218.7, 177.5)
- added J16: EPY.00.250.NTN, My Footprints:LEMO_EPY.00.250.NTN, F.Cu at (228.7, 177.5)
- added J17: EPY.00.250.NTN, My Footprints:LEMO_EPY.00.250.NTN, F.Cu at (238.7, 177.5)
- added J18: EPY.00.250.NTN, My Footprints:LEMO_EPY.00.250.NTN, F.Cu at (248.7, 177.5)
- added R117: 22, Resistor_SMD:R_1206_3216Metric, F.Cu at (173.6, 184.1)
- added R123: 22, Resistor_SMD:R_1206_3216Metric, F.Cu at (173.6, 187.4)
- added R124: 22, Resistor_SMD:R_1206_3216Metric, F.Cu at (184.0, 183.6)
- added R125: 22, Resistor_SMD:R_1206_3216Metric, F.Cu at (184.0, 186.9)
- added R126: 22, Resistor_SMD:R_1206_3216Metric, F.Cu at (195.2, 184.9)
- added R127: 22, Resistor_SMD:R_1206_3216Metric, F.Cu at (195.2, 188.2)
- added R128: 22, Resistor_SMD:R_1206_3216Metric, F.Cu at (206.9, 183.6)
- added R129: 22, Resistor_SMD:R_1206_3216Metric, F.Cu at (206.9, 186.9)
- added R130: 30, Resistor_SMD:R_0603_1608Metric, F.Cu at (166.3, 221.2)
- added U13: SN74LVC8T245PW, Package_SO:TSSOP-24_4.4x7.8mm_P0.65mm, F.Cu at (184.6, 194.5)
- added U14: SN74LVC8T245PW, Package_SO:TSSOP-24_4.4x7.8mm_P0.65mm, F.Cu at (195.3, 194.8)
- added U15: SN74LVC8T245PW, Package_SO:TSSOP-24_4.4x7.8mm_P0.65mm, F.Cu at (207.0, 194.8)
- added U16: ADR3425ARJZ, My Footprints:SOT95P280X145-6N, F.Cu at (171.8, 209.6)
- added U5: SN74LVC8T245PW, Package_SO:TSSOP-24_4.4x7.8mm_P0.65mm, F.Cu at (174.1, 194.3)
- U10: value SN74AVC8T245PW -> SN74LVC8T245PW
- moved L17 53.8 mm to (162.0, 211.1), turned to 180 degrees
- moved C44 51.2 mm to (162.0, 209.0), turned to 180 degrees
- moved C47 48.5 mm to (162.0, 206.8), turned to 180 degrees
- moved R109 42.5 mm to (300.6, 190.1)
- moved R114 42.5 mm to (301.3, 195.1)
- moved R101 42.5 mm to (301.3, 201.7)
- moved R113 42.5 mm to (301.3, 197.6)
- moved U7 42.3 mm to (163.9, 202.8), turned to 90 degrees
- moved R102 42.2 mm to (260.5, 199.4)
- moved R110 42.2 mm to (260.5, 201.9)
- moved R115 42.2 mm to (260.6, 191.9)
- moved R116 42.2 mm to (260.6, 194.4)
- moved C55 38.7 mm to (161.9, 198.6), turned to 180 degrees
- moved C61 36.2 mm to (161.9, 196.4), turned to 180 degrees
- moved R93 35.3 mm to (166.2, 198.6), turned to 0 degrees
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Connections:
- J4 pad A1: unconnected-(J4-PadA1) -> /Digital Outputs/DIGOUT0
- J4 pad A2: unconnected-(J4-PadA2) -> /Digital Outputs/DIGOUT4
- J4 pad B1: unconnected-(J4-PadB1) -> /Digital Outputs/DIGOUT1
- J4 pad B2: unconnected-(J4-PadB2) -> /Digital Outputs/DIGOUT5
- J4 pad C1: unconnected-(J4-PadC1) -> /Digital Outputs/DIGOUT2
- J4 pad C2: unconnected-(J4-PadC2) -> /Digital Outputs/DIGOUT6
- J4 pad D1: unconnected-(J4-PadD1) -> /Digital Outputs/DIGOUT3
- J4 pad D2: unconnected-(J4-PadD2) -> /Digital Outputs/DIGOUT7
- U10 pad 1: +1.8V -> +3.3V
- U10 pad 10: /DAC/dac_sdo -> unconnected-(U10-A8-Pad10)
- U10 pad 12: Net-(U10-GND-Pad12) -> GND
- U10 pad 13: Net-(U10-GND-Pad12) -> GND
- U10 pad 14: /DAC/SDO -> unconnected-(U10-B8-Pad14)
- U10 pad 16: Net-(U10-B6) -> /DAC/BIN_2SCOMP
- U10 pad 17: Net-(U10-B5) -> /DAC/CLRN
- U10 pad 18: Net-(U10-B4) -> /DAC/LDACN
- U10 pad 19: Net-(U10-B3) -> /DAC/SYNCN
- U10 pad 20: Net-(U10-B2) -> /DAC/SCLK
- U10 pad 21: Net-(U10-B1) -> /DAC/SDIN
- U10 pad 23: +3.3V -> +1.8V
- U10 pad 24: +3.3V -> +1.8V
- U10 pad 3: /DAC/SDIN -> Net-(U10-A1)
- U10 pad 4: /DAC/SCLK -> Net-(U10-A2)
- U10 pad 5: /DAC/SYNCN -> Net-(U10-A3)
- U10 pad 6: /DAC/LDACN -> Net-(U10-A4)
- U10 pad 7: /DAC/CLRN -> Net-(U10-A5)
- U10 pad 8: /DAC/BIN_2SCOMP -> Net-(U10-A6)
- U11 pad 10: Net-(U10-B4) -> Net-(U10-A4)
- U11 pad 11: Net-(U10-B5) -> Net-(U10-A5)
- U11 pad 16: /DAC/dac_sdo -> unconnected-(U11-SDO-Pad16)
- U11 pad 17: unconnected-(U11-REFIN-Pad17) -> Net-(U11-REFIN)
- U11 pad 5: Net-(U10-B6) -> Net-(U10-A6)
- U11 pad 7: Net-(U10-B3) -> Net-(U10-A3)
- U11 pad 8: Net-(U10-B2) -> Net-(U10-A2)
- U11 pad 9: Net-(U10-B1) -> Net-(U10-A1)
